File: schemes/schemes.kicad_sch (KiCad schematic)
At the start: 10 parts, among them K1 Relay_SPST-NO, K2 Relay_SPDT, M1 Вентилятор охлаждения, M2 Motor_DC, SW1 Датчик включения вентилятора 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, SW2 Включатель вентилятора охлажд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, SW3 SW_SP4T

Commit message: Add final docs
Parts:
- added M3: Motor_DC_ALT, symbol Motor:Motor_DC_ALT
- added SW4, SW5: SW_SPDT, symbol Switch:SW_SPDT
- M2: value Motor_DC -> Вентилятор отопителя
Connections:
- net GNDPWR: now also SW4.1 (A), SW5.1 (A)
- new net: M3.2 (-), SW5.2 (B)
- new net: M3.1 (+), SW4.2 (B)
- new net +BATT: SW4.3 (C), SW5.3 (C)
Other:
- note added: "2"
- note added: "3"
- note added: "5"
- note added: "6"
- note added: "Включение ЭСП"
- note added: "Переключатель ЭСП"
- note added: "Синий/Оранж"
- note added: "Чёрный"
